File: Helenowiak_elektronika/Helenowiak.sch (KiCad schematic (older format))
At the start: 19 parts

Commit message: Wszystko oprocz stm32
Parts:
- removed C?: 0.33uF, symbol Device:C
- removed U?: L7805, symbol Regulator_Linear:L7805
- added C?: 50uF, symbol Device:C
- added C?: 100uF, symbol Device:C
- added C?: 4u7, symbol Device:C
- added C? (x5): 100n, symbol Device:C
- added C?: 1u, symbol Device:C
- added CO? (x2): Czujnik_Polulu2578, symbol HelenowiakLib:CzujnikOdleglosci_Polulu2578
- added D? (x2): LED, symbol Device:LED
- added L?: 27n, symbol Device:L
- added R? (x2): 20k, symbol Device:R
- added R? (x2): 200R, symbol Device:R
- added R? (x2): 10k, symbol Device:R
- added SW? (x3): SW_DPST_x2, symbol Switch:SW_DPST_x2
- added U? (x2): CNY70, OptoDevice:Vishay_CNY70, symbol Sensor_Proximity:CNY70
- added U?: STM32F051C8Tx, Package_QFP:LQFP-48_7x7mm_P0.5mm, symbol MCU_ST_STM32F0:STM32F051C8Tx
- C?: value 0.33uF -> 10uF
- C?: value 100nF -> 10uF
Connections:
- net labels added: +7.5V, CB_out1, CB_out2, CB_out3, CO_enb1, CO_enb2, CO_enb3, CO_out1, CO_out2, CO_out3
- wire segments 96 -> 151
Other:
- note added: "Mikrokontroler STM32"
- note added: "Mosteki H / silniki / enkodery"
- note added: "Uklad zawiera diode informujaca o wykryciu obiektu"
- note added: "Uruchamianie roznych trybow testowych / taktyk"
- moved on the sheet: B?, C?, CO?, J?, M?, R?, U?

Commit message: Mechanika prawie gotowa, elektronika brak stm32
Parts:
- added RV?: R_POT, symbol Device:R_POT
Connections:
- wire segments 151 -> 163
Other:
- note added: "Wszystkie ,,puste" piny zostana odprowadzone na bok do konektorow zenskich zeby \new podpiac tam jakies diody albo dodatkowe czujniki"
- moved on the sheet: C?, L?
Changed lines of the file:
@@
 Text GLabel 4100 2500 0    50   Input ~ 0
 CO_out2
-Text GLabel 3150 3050 0    50   Output ~ 0
+Text GLabel 3150 3050 0    50   Input ~ 0
 CO_out3
 Text GLabel 2250 2400 0    50   Input ~ 0
@@
 L MCU_ST_STM32F0:STM32F051C8Tx U?
 U 1 1 606F542E
-P 8550 3350
-F 0 "U?" H 8550 1661 50  0000 C CNN
-F 1 "STM32F051C8Tx" H 8550 1570 50  0000 C CNN
-F 2 "Package_QFP:LQFP-48_7x7mm_P0.5mm" H 8050 1850 50  0001 R CNN
-F 3 "http://www.st.com/st-web-ui/static/active/en/resource/technical/document/datasheet/DM00039193.pdf" H 8550 3350 50  0001 C CNN
-	1    8550 3350
+P 8250 3200
+F 0 "U?" H 8250 1511 50  0000 C CNN
+F 1 "STM32F051C8Tx" H 8250 1420 50  0000 C CNN
+F 2 "Package_QFP:LQFP-48_7x7mm_P0.5mm" H 7750 1700 50  0001 R CNN
+F 3 "http://www.st.com/st-web-ui/static/active/en/resource/technical/document/datasheet/DM00039193.pdf" H 8250 3200 50  0001 C CNN
+	1    8250 3200
 	1    0    0    -1
 $EndComp
@@
 Wire Wire Line
 	7750 1050 8150 1050
-Wire Wire Line
-	8150 1050 8150 1450
 Connection ~ 7750 1050
-Text GLabel 10600 1050 2    50   Input ~ 0
+Text GLabel 9900 1050 2    50   Input ~ 0
 +3.3V
 $Comp
 L Device:L L?
 U 1 1 607BF2E6
-P 10300 1050
-F 0 "L?" V 10490 1050 50  0000 C CNN
-F 1 "27n" V 10399 1050 50  0000 C CNN
-F 2 "" H 10300 1050 50  0001 C CNN
-F 3 "~" H 10300 1050 50  0001 C CNN
-	1    10300 1050
+P 9600 1050
+F 0 "L?" V 9790 1050 50  0000 C CNN
+F 1 "27n" V 9699 1050 50  0000 C CNN
+F 2 "" H 9600 1050 50  0001 C CNN
+F 3 "~" H 9600 1050 50  0001 C CNN
+	1    9600 1050
 	0    -1   -1   0
 $EndComp
@@
 L Device:C C?
 U 1 1 607CCE11
-P 9450 1200
-F 0 "C?" H 9565 1246 50  0000 L CNN
-F 1 "100n" H 9565 1155 50  0000 L CNN
-F 2 "" H 9488 1050 50  0001 C CNN
-F 3 "~" H 9450 1200 50  0001 C CNN
-	1    9450 1200
+P 8750 1200
+F 0 "C?" H 8865 1246 50  0000 L CNN
+F 1 "100n" H 8865 1155 50  0000 L CNN
+F 2 "" H 8788 1050 50  0001 C CNN
+F 3 "~" H 8750 1200 50  0001 C CNN
+	1    8750 1200
 	1    0    0    -1
 $EndComp
@@
 L Device:C C?
 U 1 1 607D8702
-P 9900 1200
-F 0 "C?" H 10015 1246 50  0000 L CNN
-F 1 "1u" H 10015 1155 50  0000 L CNN
-F 2 "" H 9938 1050 50  0001 C CNN
-F 3 "~" H 9900 1200 50  0001 C CNN
-	1    9900 1200
-	1    0    0    -1
-$EndComp
-Wire Wire Line
-	10150 1050 9900 1050
-Connection ~ 9900 1050
-Wire Wire Line
-	10450 1050 10600 1050
-Wire Wire Line
-	9900 1350 9450 1350
+P 9200 1200
+F 0 "C?" H 9315 1246 50  0000 L CNN
+F 1 "1u" H 9315 1155 50  0000 L CNN
+F 2 "" H 9238 1050 50  0001 C CNN
+F 3 "~" H 9200 1200 50  0001 C CNN
+	1    9200 1200
+	1    0    0    -1
+$EndComp
+Wire Wire Line
+	9450 1050 9200 1050
+Connection ~ 9200 1050
+Wire Wire Line
+	9750 1050 9900 1050
+Wire Wire Line
+	9200 1350 8750 1350
 $Comp
 L power:GND #PWR?
 U 1 1 607FB9C7
-P 9900 1450
-F 0 "#PWR?" H 9900 1200 50  0001 C CNN
-F 1 "GND" H 9905 1277 50  0000 C CNN
-F 2 "" H 9900 1450 50  0001 C CNN
-F 3 "" H 9900 1450 50  0001 C CNN
-	1    9900 1450
-	1    0    0    -1
-$EndComp
-Wire Wire Line
-	9900 1350 9900 1450
-Connection ~ 9900 1350
-Wire Wire Line
-	9450 1050 9900 1050
-Wire Wire Line
-	9450 1050 9150 1050
-Wire Wire Line
-	9150 1050 9150 1450
-Connection ~ 9450 1050
+P 9200 1450
+F 0 "#PWR?" H 9200 1200 50  0001 C CNN
+F 1 "GND" H 9205 1277 50  0000 C CNN
+F 2 "" H 9200 1450 50  0001 C CNN
+F 3 "" H 9200 1450 50  0001 C CNN
+	1    9200 1450
+	1    0    0    -1
+$EndComp
+Wire Wire Line
+	9200 1350 9200 1450
+Connection ~ 9200 1350
+Wire Wire Line
+	8750 1050 9200 1050
+Wire Wire Line
+	8750 1050 8450 1050
+Connection ~ 8750 1050
 $Comp
 L Switch:SW_DPST_x2 SW?
@@
 Text Notes 5700 4900 0    50   ~ 10
 Uruchamianie roznych trybow testowych / taktyk
+Wire Wire Line
+	8150 1050 8150 1500
+Wire Wire Line
+	8150 1500 8250 1500
+Wire Wire Line
+	8250 1500 8250 1600
+Connection ~ 8150 1500
+Wire Wire Line
+	8150 1500 8150 1600
+Wire Wire Line
+	8250 1500 8350 1500
+Wire Wire Line
+	8350 1500 8350 1600
+Connection ~ 8250 1500
+Wire Wire Line
+	8450 1600 8450 1050
+Text Notes 7600 6000 0    50   ~ 0
+Wszystkie ,,puste" piny zostana odprowadzone na bok do konektorow zenskich zeby \new podpiac tam jakies diody albo dodatkowe czujniki
+Text GLabel 8650 5150 2    50   Input ~ 0
+GND
+Wire Wire Line
+	8150 4800 8150 4850
+Wire Wire Line
+	8150 4850 8250 4850
+Wire Wire Line
+	8250 4850 8250 4800
+Wire Wire Line
+	8250 4850 8350 4850
+Wire Wire Line
+	8350 4850 8350 4800
+Connection ~ 8250 4850
+Wire Wire Line
+	8250 4850 8250 5150
+Wire Wire Line
+	8250 5150 8650 5150
+Text GLabel 6500 2450 0    50   Input ~ 0
+CO_out1
+Text GLabel 6500 2350 0    50   Input ~ 0
+CO_enb1
+Text GLabel 6500 2650 0    50   Input ~ 0
+CO_out2
+Text GLabel 6500 2550 0    50   Input ~ 0
+CO_enb2
+Text GLabel 6500 2850 0    50   Input ~ 0
+CO_out3
+Text GLabel 6500 2750 0    50   Input ~ 0
+CO_enb3
+Text GLabel 6400 2150 0    50   Input ~ 0
+BT_RX
+Text GLabel 6400 2250 0    50   Input ~ 0
+BT_TX
+Text GLabel 6750 2950 0    50   Input ~ 0
+OUTA_EnkoderL
+Text GLabel 6750 3050 0    50   Input ~ 0
+OUTB_EnkoderL
+Text GLabel 6350 3350 0    50   Input ~ 0
+L_IN1
+Text GLabel 6350 3250 0    50   Input ~ 0
+L_IN2
+Text GLabel 6400 3150 0    50   Input ~ 0
+L_PWM
+Text GLabel 6350 3850 0    50   Input ~ 0
+R_IN1
+Text GLabel 6350 3750 0    50   Input ~ 0
+R_IN2
+Text GLabel 6400 3650 0    50   Input ~ 0
+R_PWM
+Text GLabel 6700 3450 0    50   Input ~ 0
+OUTA_EnkoderR
+Text GLabel 6700 3550 0    50   Input ~ 0
+OUTB_EnkoderR
+Text GLabel 6450 3950 0    50   Input ~ 0
+CB_out1
+Text GLabel 6450 4050 0    50   Input ~ 0
+CB_out2
+Text GLabel 6450 4150 0    50   Input ~ 0
+CB_out3
+$Comp
+L Device:R_POT RV?
+U 1 1 60628E41
+P 2300 7100
+F 0 "RV?" H 2231 7146 50  0000 R CNN
+F 1 "R_POT" H 2231 7055 50  0000 R CNN
+F 2 "" H 2300 7100 50  0001 C CNN
+F 3 "~" H 2300 7100 50  0001 C CNN
+	1    2300 7100
+	1    0    0    -1
+$EndComp
 $EndSCHEMATC

Commit message: Mechanika prawie gotowa, elektronika brak stm32
Parts:
- removed CO?: Czujnik_Polulu2578, symbol HelenowiakLib:CzujnikOdleglosci_Polulu2578
- removed R?: 20k, symbol Device:R
- removed R?: 200R, symbol Device:R
- removed U?: CNY70, OptoDevice:Vishay_CNY70, symbol Sensor_Proximity:CNY70
Connections:
- net labels removed: CB_out3, CO_enb3, CO_out3
- wire segments 163 -> 151
Other:
- moved on the sheet: CO?, R?, U?

Commit message: New stm32
Parts:
- removed H? (x2): TB6612FNG, symbol HelenowiakLib:TB6612FNG
- removed RV?: R_POT, symbol Device:R_POT
- removed SW? (x2): SW_DPST_x2, symbol Switch:SW_DPST_x2
- removed U?: STM32F051C8Tx, Package_QFP:LQFP-48_7x7mm_P0.5mm, symbol MCU_ST_STM32F0:STM32F051C8Tx
- added C? (x4): 0.1uF, symbol Device:C
- added C?: 100n, symbol Device:C
- added R?: 100k, symbol Device:R
- added SW?: SW_MEC_5G, symbol Switch:SW_MEC_5G
- added U? (x2): DRV8835DSSR, DSS0012A, symbol HelenowiakLib:DRV8835DSSR
- added U?: STM32F105RCTx, Package_QFP:LQFP-64_10x10mm_P0.5mm, symbol MCU_ST_STM32F1:STM32F105RCTx
- L?: value 27n -> 10u
- R? (x2): value 10k -> 220R
Connections:
- net labels added: L_MODE, R_MODE, Reset
- net labels removed: L_PWM, R_PWM
- wire segments 151 -> 148
Other:
- note removed: "Uruchamianie roznych trybow testowych / taktyk"
- moved on the sheet: C?, D?, J?, L?, M?, R?, U?

Commit message: New pinout
Parts:
- removed D?: LED, symbol Device:LED
- removed R?: 220R, symbol Device:R
- added C?: 10uF, symbol Device:C
- added C? (x2): 100n, symbol Device:C
- added D? (x2): LED, symbol Device:LED
- added Q?: BS170, Package_TO_SOT_THT:TO-92_Inline, symbol Transistor_FET:BS170
- added R?: 1K, symbol Device:R
- added R? (x3): 100k, symbol Device:R
- added R?: 47k, symbol Device:R
- added R? (x2): 220R, symbol Device:R
- added SW? (x2): SW_MEC_5G, symbol Switch:SW_MEC_5G
Connections:
- net +3.3V: now also R?.1, R?.1
- net CO_enb1: now also U?.33 (PB12)
- net CO_enb2: now also U?.34 (PB13)
- net CO_out1: now also U?.35 (PB14)
- net CO_out2: now also U?.36 (PB15)
- net GND: now also U?.60 (BOOT0), C?.2, C?.2, C?.2, D?.1 (K), D?.1 (K), Q?.1 (D), R?.2; no longer J?.1 (Pin_1)
- net L_MODE: now also U?.24 (PC4)
- net OUTA_EnkoderL: now also U?.41 (PA8)
- net OUTA_EnkoderR: now also U?.50 (PA15)
- net OUTB_EnkoderL: now also U?.42 (PA9)
- net OUTB_EnkoderR: now also U?.55 (PB3)
- net R_MODE: now also U?.25 (PC5)
- net LED1: now reaches R?.2
- net Battery_V: now reaches U?.21 (PA5)
- net Battery_V: now also C?.1, R?.1, R?.2
- net PWM_L_IN1: now reaches U?.22 (PA6)
- net PWM_L_IN2: now reaches U?.23 (PA7)
- net PWM_R_IN1: now reaches U?.26 (PB0)
- net PWM_R_IN2: now reaches U?.27 (PB1)
- net +7.5V renamed +7.4V
- net +7.4V: now also R?.1, R?.1
- new net: J?.1 (Pin_1), Q?.3 (S)
- new net: Q?.2 (G), R?.2
- new net: D?.2 (A), R?.1 (x2)
- new net: SW?.1 (A), SW?.2 (A) (x2)
- new net Button1: C?.1, R?.2, SW?.3 (B), SW?.4 (B)
- new net Button2: C?.1, R?.2, SW?.3 (B), SW?.4 (B)
- new net LED2: R?.2
- new net LED3: R?.2
Other:
- note added: "Czujnik bieli"
- note added: "Zasilanie, zabezpieczenie przed odwrotna polaryzacja, pomiar napiecia na baterii\n\n"
- note removed: "Detektor bieli"
- note removed: "Uklad zawiera diode informujaca o wykryciu obiektu"
- note removed: "Zasilanie\n"
- moved on the sheet: B?, C?, CO?, D?, J?, R?, SW?, SW?A, U?

Commit message: Finished eschema
Parts:
- removed C? (x2): 100n, symbol Device:C
- removed R? (x2): 100k, symbol Device:R
- removed SW? (x2): SW_MEC_5G, symbol Switch:SW_MEC_5G
- added C16, C19, C8: 100n, symbol Device:C
- added D4: LED, symbol Device:LED
- added J2: Conn_01x05_Female, symbol Connector:Conn_01x05_Female
- added J3: Conn_01x04_Female, symbol Connector:Conn_01x04_Female
- added J5: Conn_01x08_Female, symbol Connector:Conn_01x08_Female
- added R13: 220R, symbol Device:R
- added R5, R7, R9: 100R, symbol Device:R
- added R6, R8: 4k7, symbol Device:R
- added SW3, SW4: SW_MEC_5G, symbol Switch:SW_MEC_5G
- CO1, CO2: renamed from CO?; symbol HelenowiakLib:CzujnikOdleglosci_Polulu2578 -> Helenowiak-rescue:CzujnikOdleglosci_Polulu2578-HelenowiakLib
- R4: renamed from R?; value 100k -> 4k7
- gave numbers to parts that had none: 48
Connections:
- net +3.3V: now also C8.1, J2.2 (Pin_2), J3.1 (Pin_1), R6.1, R8.1
- net +5.0V: now also CO1.~ (VDD), CO2.~ (VDD); no longer CO1.3 (VDD), CO2.3 (VDD)
- net Button1: now also U3.37 (PC6), C16.2, R6.2, SW3.3 (B), SW3.4 (B)
- net Button2: now also U3.38 (PC7), C19.2, R8.2, SW4.3 (B), SW4.4 (B)
- net CO_enb1: now also CO1.~ (VDD); no longer CO1.1 (Enable)
- net CO_enb2: now also CO2.~ (VDD); no longer CO2.1 (Enable)
- net CO_out1: now also CO1.~ (VDD); no longer CO1.2 (OUT)
- net CO_out2: now also CO2.~ (VDD); no longer CO2.2 (OUT)
- net GND: now also CO1.~ (VDD), CO2.~ (VDD), C8.2, D4.1 (K), J2.1 (Pin_1), J3.2 (Pin_2), R5.1, R7.1, R9.1, SW3.1 (A), SW3.2 (A), SW4.1 (A), SW4.2 (A); no longer C15.2, CO1.4 (GND), CO2.4 (GND)
- net LED1: now also U3.8 (PC0)
- net LED2: now also U3.9 (PC1)
- net LED3: now also U3.10 (PC2)
- net Reset: now also C15.2, J2.3 (Pin_3); no longer C15.1
- net LED4: now reaches U3.11 (PC3)
- net LED4: now also R13.2
- net at U3.2 (PC13): now also J5.3 (Pin_3)
- net Extra_TX: now reaches U3.29 (PB10)
- net Extra_TX: now also J3.3 (Pin_3)
- net at U3.3 (PC14): now also J5.2 (Pin_2)
- net Extra_RX: now reaches U3.30 (PB11)
- net Extra_RX: now also J3.4 (Pin_4)
- net at U3.39 (PC8): now also J5.8 (Pin_8)
- net at U3.4 (PC15): now also J5.1 (Pin_1)
- net at U3.40 (PC9): now also J5.7 (Pin_7)
- net SYS_JTMS-SWDIO: now reaches U3.46 (PA13)
- net SYS_JTMS-SWDIO: now also J2.4 (Pin_4)
- net SYS_JTCK-SWCLK: now reaches U3.49 (PA14)
- net SYS_JTCK-SWCLK: now also J2.5 (Pin_5)
- net at U3.51 (PC10): now also J5.6 (Pin_6)
- net at U3.52 (PC11): now also J5.5 (Pin_5)
- net at U3.53 (PC12): now also J5.4 (Pin_4)
- new net: C15.1, R5.2
- new net: C16.1, R7.2
- new net: C19.1, R9.2
- new net: D4.2 (A), R13.1
- no-connect marks 6 -> 19
Other:
- note added: "Dodatkowy UART"
- note added: "Programator"
- moved on the sheet: C15, D1, D2, D3, R10, R11, R12, R4, SW2

Commit message: Etap II
Parts:
- removed M1: MotorL, symbol Helenowiak-rescue:Motor_DC-Motor
- removed M2: MotorR, symbol Helenowiak-rescue:Motor_DC-Motor
- removed SW1: SW_DPST_x2, symbol Switch:SW_DPST_x2
- added C22, C24: 100nF, Capacitors_SMD:C_0603, symbol Device:C
- added C23: 10uF, Capacitors_SMD:C_0603, symbol Device:C
- added SW1: SW_SPDT, Connector_PinSocket_2.54mm:PinSocket_1x03_P2.54mm_Vertical, symbol Switch:SW_SPDT
- B1: value BT05 -> HC-06; footprint (none) -> Connector_PinSocket_2.54mm:PinSocket_1x06_P2.54mm_Vertical
- C1, C11, C14, C15, C16, C17, C18, C19, C2, C20, C21, C3, C4, C5, C6, C7, C8, C9: footprint (none) -> Capacitors_SMD:C_0603
- C10: value 50uF -> 100nF; footprint (none) -> Capacitors_SMD:C_0603
- C12: value 100uF -> 10uF; footprint (none) -> Capacitors_SMD:C_0603
- C13: value 10uF -> 100nF; footprint (none) -> Capacitors_SMD:C_0603
- CO1, CO2: footprint (none) -> Connector_PinSocket_2.54mm:PinSocket_1x04_P2.54mm_Vertical; symbol Helenowiak-rescue:CzujnikOdleglosci_Polulu2578-HelenowiakLib -> HelenowiakLib:CzujnikOdleglosci_Polulu2578
- D1, D2, D3, D4: footprint (none) -> LED_SMD:LED_0603_1608Metric
- J1: footprint (none) -> Connector_PinSocket_2.54mm:PinSocket_1x02_P2.54mm_Vertical
- J2: value Conn_01x05_Female -> Conn_programator; footprint (none) -> Connector_PinSocket_2.54mm:PinSocket_1x05_P2.54mm_Vertical
- J3: value Conn_01x04_Female -> Conn_extraUART; footprint (none) -> Connector_PinSocket_2.54mm:PinSocket_1x04_P2.54mm_Vertical
- J4, J6: footprint (none) -> Connector_PinSocket_2.54mm:PinSocket_1x06_P2.54mm_Vertical
- J5: value Conn_01x08_Female -> freePins; footprint (none) -> Connector_PinSocket_2.54mm:PinSocket_1x08_P2.54mm_Vertical
- L1: footprint (none) -> Inductors_SMD:L_0603
- R1, R10, R11, R12, R13, R14, R15, R16, R17, R2, R3, R4, R5, R6, R7, R8, R9: footprint (none) -> Resistor_SMD:R_0603_1608Metric
- SW2: value SW_MEC_5G -> Reset_button; footprint (none) -> footprints_helenowiak:button_mono
- SW3: value SW_MEC_5G -> button1; footprint (none) -> footprints_helenowiak:button_mono
- SW4: value SW_MEC_5G -> button2; footprint (none) -> footprints_helenowiak:button_mono
- U1: footprint (none) -> Package_TO_SOT_THT:TO-220-3_Vertical
- U4: footprint DSS0012A -> Housings_SON:WSON-12-1EP_3x2mm_Pitch0.5mm
- U5: footprint DSS0012A -> Package_SON:WSON-12-1EP_3x2mm_P0.5mm_EP1x2.65
Connections:
- net L_IN1 is gone; now on net PWM_L_IN1: U4.10 (AIN1_APHASE), U4.8 (BIN1_BPHASE)
- net L_IN2 is gone; now on net PWM_L_IN2: U4.7 (BIN2_BENBL), U4.9 (AIN2_AENBL)
- net CO_enb1: now also CO1.1 (Enable); no longer CO1.~ (VDD)
- net CO_enb2: now also CO2.1 (Enable); no longer CO2.~ (VDD)
- net CO_out1: now also CO1.2 (OUT); no longer CO1.~ (VDD)
- net CO_out2: now also CO2.2 (OUT); no longer CO2.~ (VDD)
- net GND: now also CO1.4 (GND), CO2.4 (GND), C22.2, C23.2, C24.2; no longer CO1.~ (VDD), CO2.~ (VDD)
- net PWM_R_IN1: now also U5.10 (AIN1_APHASE), U5.8 (BIN1_BPHASE)
- net PWM_R_IN2: now also U5.7 (BIN2_BENBL)
- net at J1.2 (Pin_2): now also SW1.2 (B)
- net +3.3V renamed +3V3
- net +3V3: now also C24.1; no longer B1.5 (VCC), J3.1 (Pin_1)
- net +5.0V renamed +5V
- net +5V: now also B1.5 (VCC), CO1.3 (VDD), CO2.3 (VDD), J3.1 (Pin_1), C22.1, C23.1; no longer CO1.~ (VDD), CO2.~ (VDD)
- net +7.4V renamed +7.5V
- net +7.5V: now also SW1.3 (C)
- removed net R_IN1: U5.10 (AIN1_APHASE), U5.7 (BIN2_BENBL), U5.8 (BIN1_BPHASE)
- no-connect marks 19 -> 17
Other:
- note removed: "Wszystkie ,,puste" piny zostana odprowadzone na bok do konektorow zenskich zeby \new podpiac tam jakies diody albo dodatkowe czujniki"
- moved on the sheet: C13, C14, U2

Commit message: PCB 75%
Parts:
- CO1, CO2: symbol HelenowiakLib:CzujnikOdleglosci_Polulu2578 -> Connector:Conn_01x04_Female
- J1: value Conn_01x02_Female -> Vin
- SW2, SW3, SW4: symbol Switch:SW_MEC_5G -> Switch:SW_Push
Connections:
- net +5V: no longer U3.14 (PA0), U3.16 (PA2)
- net Button1: now also SW3.2; no longer SW3.3 (B), SW3.4 (B)
- net Button2: now also SW4.2; no longer SW4.3 (B), SW4.4 (B)
- net GND: no longer SW2.2 (A), SW3.2 (A), SW4.2 (A)
- net Reset: now also SW2.2; no longer SW2.3 (B), SW2.4 (B)
- net CB_out1: now reaches R15.2, U6.3 (C)
- net CB_out1: now also U3.14 (PA0)
- net CB_out2: now reaches R17.2, U7.3 (C)
- net CB_out2: now also U3.16 (PA2)
Changed lines of the file:
@@
 P 650 1500
 F 0 "J1" H 678 1476 50  0000 L CNN
-F 1 "Conn_01x02_Female" H 678 1385 50  0000 L CNN
+F 1 "Vin" H 678 1385 50  0000 L CNN
 F 2 "Connector_PinSocket_2.54mm:PinSocket_1x02_P2.54mm_Vertical" H 650 1500 50  0001 C CNN
 F 3 "~" H 650 1500 50  0001 C CNN
@@
 $EndComp
 $Comp
-L Regulator_Linear:LD1117S33TR_SOT223 U2
-U 1 1 60505D10
-P 4350 1050
-F 0 "U2" H 4350 1292 50  0000 C CNN
-F 1 "LD1117S33TR_SOT223" H 4350 1201 50  0000 C CNN
-F 2 "Package_TO_SOT_SMD:SOT-223-3_TabPin2" H 4350 1250 50  0001 C CNN
-F 3 "http://www.st.com/st-web-ui/static/active/en/resource/technical/document/datasheet/CD00000544.pdf" H 4450 800 50  0001 C CNN
-	1    4350 1050
-	1    0    0    -1
-$EndComp
-$Comp
 L Device:C C13
 U 1 1 6050FAF6
@@
 $EndComp
 $Comp
-L HelenowiakLib:CzujnikOdleglosci_Polulu2578 CO1
+L Connector:Conn_01x04_Female CO1
 U 1 1 6055C9E9
-P 2700 2900
-F 0 "CO1" H 2878 2951 50  0000 L CNN
-F 1 "Czujnik_Polulu2578" H 2878 2860 50  0000 L CNN
-F 2 "Connector_PinSocket_2.54mm:PinSocket_1x04_P2.54mm_Vertical" H 2450 2850 50  0001 C CNN
-F 3 "" H 2450 2850 50  0001 C CNN
-	1    2700 2900
+P 2600 2850
+F 0 "CO1" H 2778 2901 50  0000 L CNN
+F 1 "Czujnik_Polulu2578" H 2778 2810 50  0000 L CNN
+F 2 "Connector_PinSocket_2.54mm:PinSocket_1x04_P2.54mm_Vertical" H 2350 2800 50  0001 C CNN
+F 3 "" H 2350 2800 50  0001 C CNN
+	1    2600 2850
 	1    0    0    -1
 $EndComp
@@
 NoConn ~ 900  3250
 $Comp
-L Regulator_Linear:LM1117-5.0 U1
-U 1 1 604A7886
-P 2800 1700
-F 0 "U1" H 2800 1942 50  0000 C CNN
-F 1 "LM1117-5.0" H 2800 1851 50  0000 C CNN
-F 2 "Package_TO_SOT_THT:TO-220-3_Vertical" H 2800 1700 50  0001 C CNN
-F 3 "http://www.ti.com/lit/ds/symlink/lm1117.pdf" H 2800 1700 50  0001 C CNN
-	1    2800 1700
-	1    0    0    -1
-$EndComp
-$Comp
 L Device:C C10
 U 1 1 60533C27
@@
 Bluetooth
 $Comp
-L HelenowiakLib:CzujnikOdleglosci_Polulu2578 CO2
+L Connector:Conn_01x04_Female CO2
 U 1 1 605979D7
-P 4550 2900
-F 0 "CO2" H 4728 2951 50  0000 L CNN
-F 1 "Czujnik_Polulu2578" H 4728 2860 50  0000 L CNN
-F 2 "Connector_PinSocket_2.54mm:PinSocket_1x04_P2.54mm_Vertical" H 4300 2850 50  0001 C CNN
-F 3 "" H 4300 2850 50  0001 C CNN
-	1    4550 2900
+P 4450 2850
+F 0 "CO2" H 4628 2901 50  0000 L CNN
+F 1 "Czujnik_Polulu2578" H 4628 2810 50  0000 L CNN
+F 2 "Connector_PinSocket_2.54mm:PinSocket_1x04_P2.54mm_Vertical" H 4200 2800 50  0001 C CNN
+F 3 "" H 4200 2800 50  0001 C CNN
+	1    4450 2850
 	1    0    0    -1
 $EndComp
@@
 	4650 6900 4650 6950
 Connection ~ 3950 6900
-Text GLabel 4850 6900 2    50   Output ~ 0
+Text GLabel 4750 7300 2    50   Output ~ 0
 CB_out2
-Wire Wire Line
-	4650 6900 4850 6900
-Connection ~ 4650 6900
 Connection ~ 2250 1700
 Wire Wire Line
@@
 Wire Wire Line
 	1550 7650 2150 7650
-Connection ~ 2250 6900
-Wire Wire Line
-	2250 6900 2450 6900
-Text GLabel 2450 6900 2    50   Output ~ 0
+Text GLabel 2350 7300 2    50   Output ~ 0
 CB_out1
 Connection ~ 1550 6900
@@
 	9250 5100 9250 5300
 $Comp
-L Switch:SW_MEC_5G SW2
-U 1 1 60BC18A3
-P 6150 1900
-F 0 "SW2" H 6150 2185 50  0000 C CNN
-F 1 "Reset_button" H 6150 2094 50  0000 C CNN
-F 2 "footprints_helenowiak:button_mono" H 6150 2100 50  0001 C CNN
-F 3 "http://www.apem.com/int/index.php?controller=attachment&id_attachment=488" H 6150 2100 50  0001 C CNN
-	1    6150 1900
-	1    0    0    -1
-$EndComp
-$Comp
 L Device:C C15
 U 1 1 60BD1750
@@
 Wire Wire Line
 	1600 1400 1600 1700
-Text GLabel 2250 1350 0    50   Output ~ 0
-Battery_V
 Text Notes 600  750  0    50   ~ 10
 Zasilanie, zabezpieczenie przed odwrotna polaryzacja, pomiar napiecia na baterii\n\n
@@
 Connection ~ 6600 1900
 $Comp
-L Switch:SW_MEC_5G SW3
+L Switch:SW_Push SW3
 U 1 1 608F1124
 P 6150 3000
@@
 Connection ~ 6600 3000
 $Comp
-L Switch:SW_MEC_5G SW4
+L Switch:SW_Push SW4
 U 1 1 608FA127
 P 6150 4050
@@
 	1    0    0    -1
 $EndComp
-Connection ~ 1250 1400
 Wire Wire Line
 	850  1300 850  1400
-NoConn ~ 1250 1200
 Wire Wire Line
 	3100 1700 3200 1700
@@
 Wire Wire Line
 	10850 900  10850 950
+$Comp
+L Switch:SW_Push SW2
+U 1 1 60BC18A3
+P 6150 1900
+F 0 "SW2" H 6150 2185 50  0000 C CNN
+F 1 "Reset_button" H 6150 2094 50  0000 C CNN
+F 2 "footprints_helenowiak:button_mono" H 6150 2100 50  0001 C CNN
+F 3 "http://www.apem.com/int/index.php?controller=attachment&id_attachment=488" H 6150 2100 50  0001 C CNN
+	1    6150 1900
+	1    0    0    -1
+$EndComp
+NoConn ~ 1250 1200
+Text GLabel 2250 1350 0    50   Output ~ 0
+Battery_V
+$Comp
+L Regulator_Linear:LM1117-5.0 U1
+U 1 1 604A7886
+P 2800 1700
+F 0 "U1" H 2800 1942 50  0000 C CNN
+F 1 "LM1117-5.0" H 2800 1851 50  0000 C CNN
+F 2 "Package_TO_SOT_THT:TO-220-3_Vertical" H 2800 1700 50  0001 C CNN
+F 3 "http://www.ti.com/lit/ds/symlink/lm1117.pdf" H 2800 1700 50  0001 C CNN
+	1    2800 1700
+	1    0    0    -1
+$EndComp
+$Comp
+L Regulator_Linear:LD1117S33TR_SOT223 U2
+U 1 1 60505D10
+P 4350 1050
+F 0 "U2" H 4350 1292 50  0000 C CNN
+F 1 "LD1117S33TR_SOT223" H 4350 1201 50  0000 C CNN
+F 2 "Package_TO_SOT_SMD:SOT-223-3_TabPin2" H 4350 1250 50  0001 C CNN
+F 3 "http://www.st.com/st-web-ui/static/active/en/resource/technical/document/datasheet/CD00000544.pdf" H 4450 800 50  0001 C CNN
+	1    4350 1050
+	1    0    0    -1
+$EndComp
+Connection ~ 1250 1400
+Wire Wire Line
+	2250 7300 2350 7300
+Connection ~ 2250 7300
+Wire Wire Line
+	4650 7300 4750 7300
+Connection ~ 4650 7300
 $EndSCHEMATC
