File: Helenowiak_elektronika/Helenowiak.sch (KiCad schematic (older format))
At the start: 67 parts, among them J1 Vin, J2 Conn_programator, J3 Conn_extraUART, J4 EnkoderL, J5 freePins, J6 EnkoderR, Q1 BS170, SW1 SW_SPDT, SW2 Reset_button, SW3 button1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

Commit message: Przed wylaniem masy
Parts:
- removed J5: freePins, Connector_PinSocket_2.54mm:PinSocket_1x08_P2.54mm_Vertical, symbol Connector:Conn_01x08_Female
Changed lines of the file:
@@
 Text GLabel 9950 3450 2    50   Input ~ 0
 PWM_R_IN2
-Text GLabel 8550 3850 0    50   Output ~ 0
-R_MODE
 Text GLabel 9950 3150 2    50   Input ~ 0
 OUTA_EnkoderR
@@
 Text GLabel 6600 4350 2    50   Input ~ 0
 Button2
-Text GLabel 8550 3950 0    50   Input ~ 0
-Button1
-Text GLabel 8550 4050 0    50   Input ~ 0
-Button2
 Text GLabel 8550 3350 0    50   Output ~ 0
 LED1
@@
 Text GLabel 8550 3650 0    50   Output ~ 0
 LED4
-$Comp
-L Connector:Conn_01x08_Female J5
-U 1 1 609E65DA
-P 7650 4550
-F 0 "J5" H 7542 3925 50  0000 C CNN
-F 1 "freePins" H 7542 4016 50  0000 C CNN
-F 2 "Connector_PinSocket_2.54mm:PinSocket_1x08_P2.54mm_Vertical" H 7650 4550 50  0001 C CNN
-F 3 "~" H 7650 4550 50  0001 C CNN
-	1    7650 4550
-	-1   0    0    1
-$EndComp
-Wire Wire Line
-	8550 4150 7850 4150
-Wire Wire Line
-	8550 4250 7850 4250
-Wire Wire Line
-	7850 4350 8550 4350
-Wire Wire Line
-	8550 4450 7850 4450
-Wire Wire Line
-	7850 4550 8550 4550
-Wire Wire Line
-	8550 4650 7850 4650
-Wire Wire Line
-	7850 4750 8550 4750
-Wire Wire Line
-	8550 4850 7850 4850
 NoConn ~ 9950 1950
 NoConn ~ 9950 2050
@@
 Wire Wire Line
 	1450 5750 1450 6050
-Wire Wire Line
-	1400 5850 1350 5850
 $Comp
 L power:+5V #PWR0119
@@
 	4650 7300 4750 7300
 Connection ~ 4650 7300
+Text GLabel 8550 4050 0    50   Input ~ 0
+Button2
+Text GLabel 8550 3950 0    50   Input ~ 0
+Button1
+Text GLabel 8550 3850 0    50   Output ~ 0
+R_MODE
+Wire Wire Line
+	1400 5850 1350 5850
 $EndSCHEMATC

Commit message: PCB zamowione
Connections:
- net PWM_R_IN2: now also U5.9 (AIN2_AENBL)
Changed lines of the file:
@@
 R_MODE
 Wire Wire Line
-	1400 5850 1350 5850
+	1350 5850 1500 5850
 $EndSCHEMATC
