File: Helenowiak_elektronika/Helenowiak.kicad_pcb (KiCad board)
At the start: 2 copper layers, 86 x 35 mm, 67 parts, among them J1 Conn_01x02_Female, J2 Conn_programator, J3 Conn_extraUART, J4 EnkoderL, J5 freePins, J6 EnkoderR, Q1 BS170, SW1 SW_SPDT, SW2 Reset_button, SW3 button1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

Commit message: PCB 75%
Parts:
- J1: value Conn_01x02_Female -> Vin
- moved C10 119.6 mm to (80.2, 153.1), turned to 90 degrees
- moved R14 118.9 mm to (72.8, 130.2)
- moved C22 117.9 mm to (85.3, 137.8), turned to 270 degrees
- moved C12 117.1 mm to (80.0, 137.9), turned to 270 degrees
- moved C13 114.7 mm to (80.0, 142.3), turned to 270 degrees
- moved C23 112.4 mm to (85.3, 141.8), turned to 270 degrees
- moved C11 112.2 mm to (84.7, 153.1), turned to 90 degrees
- moved R2 109.1 mm to (113.7, 140.3)
- moved C19 104.0 mm to (141.8, 149.1), turned to 180 degrees
- moved C7 103.9 mm to (118.8, 144.6)
- moved C24 103.5 mm to (105.2, 140.3)
- moved R3 101.0 mm to (88.3, 153.1), turned to 90 degrees
- moved C15 99.7 mm to (150.4, 149.1)
- moved C9 98.1 mm to (109.6, 140.3)
- moved C20 95.1 mm to (119.2, 151.2)
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Connections:
- B1 pad 5: CB_out1 -> +5V
- C12 pad 1: CB_out1 -> +5V
- C13 pad 1: CB_out1 -> +5V
- C22 pad 1: CB_out1 -> +5V
- C23 pad 1: CB_out1 -> +5V
- CO1 pad 3: CB_out1 -> +5V
- CO2 pad 3: CB_out1 -> +5V
- J3 pad 1: CB_out1 -> +5V
- J4 pad 3: CB_out1 -> +5V
- J6 pad 3: CB_out1 -> +5V
- R14 pad 1: CB_out1 -> +5V
- R15 pad 1: CB_out1 -> +5V
- R15 pad 2: Net-(R15-Pad2) -> CB_out1
- R16 pad 1: CB_out1 -> +5V
- R17 pad 1: CB_out1 -> +5V
- R17 pad 2: Net-(R17-Pad2) -> CB_out2
- SW2 pad 2: GND -> Reset
- SW3 pad 2: GND -> Button1
- SW4 pad 2: GND -> Button2
- U1 pad 2: CB_out1 -> +5V
- U2 pad 3: CB_out1 -> +5V
- U3 pad 16: CB_out1 -> CB_out2
- U6 pad 3: Net-(R15-Pad2) -> CB_out1
- U7 pad 3: Net-(R17-Pad2) -> CB_out2
Routing:
- net +3V3: track 0.00 -> 84.9 mm
- net +5V: track 0.00 -> 80.0 mm
- net +7.5V: track 0.00 -> 27.1 mm
- net Net-(C15-Pad1): track 0.00 -> 14.8 mm
- net Net-(R16-Pad2): track 0.00 -> 11.1 mm
- net Net-(J1-Pad2): track 0.00 -> 10.7 mm
- net Net-(R14-Pad2): track 0.00 -> 9.73 mm
- net CB_out2: track 0.00 -> 5.71 mm
- net Reset: track 0.00 -> 5.69 mm
- net Net-(Q1-Pad2): track 0.00 -> 5.66 mm
- net CB_out1: track 0.00 -> 5.41 mm
- net Net-(J1-Pad1): track 0.00 -> 3.68 mm
Other:
- board size 86 x 35 mm -> 88 x 40 mm
- net class Default: trace_width 0.25 -> 1
- net class Zasilanie added: clearance 0.2, trace_width 1.5, via_dia 0.8, via_drill 0.4

Commit message: Przed wylaniem masy
Parts:
- removed J5: freePins, Connector_PinSocket_2.54mm:PinSocket_1x08_P2.54mm_Vertical
- C1, C2, C3, C4, C5, C6, C7, C8, L1, U3, U6, U7: moved to B.Cu
- moved C1 32.7 mm to (105.5, 141.1), turned to 270 degrees
- moved C2 32.6 mm to (105.5, 137.9), turned to 270 degrees
- moved L1 32.4 mm to (105.5, 144.1), turned to 270 degrees
- moved C3 19.7 mm to (105.8, 146.4), turned to 180 degrees
- moved R1 19.3 mm to (98.0, 147.0)
- moved C8 17.9 mm to (121.2, 146.6)
- moved U3 14.6 mm to (113.8, 140.1), turned to 0 degrees
- moved R2 13.4 mm to (100.5, 142.8)
- moved C17 11.4 mm to (113.9, 152.6), turned to 90 degrees
- moved C7 11.0 mm to (108.3, 147.9), turned to 180 degrees
- moved C20 10.9 mm to (130.0, 152.7), turned to 90 degrees
- moved C9 9.23 mm to (103.2, 147.0)
- moved C4 9.02 mm to (110.8, 130.6), turned to 180 degrees
- moved C5 7.63 mm to (117.2, 130.6), turned to 180 degrees
- moved C24 6.70 mm to (100.5, 135.5)
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Connections:
- B1 pad 1: Net-(B1-Pad1) -> (no net)
- B1 pad 6: Net-(B1-Pad6) -> (no net)
- SW1 pad 1: Net-(SW1-Pad1) -> (no net)
- U3 pad 15: Net-(U3-Pad15) -> (no net)
- U3 pad 17: Net-(U3-Pad17) -> (no net)
- U3 pad 2: Net-(J5-Pad3) -> (no net)
- U3 pad 20: Net-(U3-Pad20) -> (no net)
- U3 pad 28: Net-(U3-Pad28) -> (no net)
- U3 pad 3: Net-(J5-Pad2) -> (no net)
- U3 pad 39: Net-(J5-Pad8) -> (no net)
- U3 pad 4: Net-(J5-Pad1) -> (no net)
- U3 pad 40: Net-(J5-Pad7) -> (no net)
- U3 pad 43: Net-(U3-Pad43) -> (no net)
- U3 pad 44: Net-(U3-Pad44) -> (no net)
- U3 pad 45: Net-(U3-Pad45) -> (no net)
- U3 pad 5: Net-(U3-Pad5) -> (no net)
- U3 pad 51: Net-(J5-Pad6) -> (no net)
- U3 pad 52: Net-(J5-Pad5) -> (no net)
- U3 pad 53: Net-(J5-Pad4) -> (no net)
- U3 pad 54: Net-(U3-Pad54) -> (no net)
- U3 pad 56: Net-(U3-Pad56) -> (no net)
- U3 pad 57: Net-(U3-Pad57) -> (no net)
- U3 pad 6: Net-(U3-Pad6) -> (no net)
- U3 pad 61: Net-(U3-Pad61) -> (no net)
- U3 pad 62: Net-(U3-Pad62) -> (no net)
- U5 pad 9: Net-(U5-Pad9) -> (no net)
Routing:
- net +5V: track 80.0 -> 180.5 mm, vias 0 -> 1
- net Reset: track 5.69 -> 97.1 mm, vias 0 -> 4
- net LED3: track 0.00 -> 76.0 mm, vias 0 -> 5
- net CB_out2: track 5.71 -> 75.0 mm, vias 0 -> 2
- net CO_out1: track 0.00 -> 68.8 mm, vias 0 -> 2
- net LED4: track 0.00 -> 65.3 mm, vias 0 -> 1
- net +3V3: track 84.9 -> 141.2 mm, vias 0 -> 8
- net CO_enb1: track 0.00 -> 55.3 mm, vias 0 -> 2
- net BT_TX: track 0.00 -> 53.0 mm
- net Extra_TX: track 0.00 -> 51.4 mm, vias 0 -> 2
- net OUTA_EnkoderL: track 0.00 -> 50.4 mm
- net Extra_RX: track 0.00 -> 49.1 mm, vias 0 -> 2
- net OUTB_EnkoderL: track 0.00 -> 46.4 mm
- net CB_out1: track 5.41 -> 48.5 mm
- net BT_RX: track 0.00 -> 43.0 mm
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Other:
- outline, holes or cut-outs redrawn
- net class Default: clearance 0.2 -> 0.15; trace_width 1 -> 0.25
- net class Zasilanie: clearance 0.2 -> 0.5; trace_width 1.5 -> 0.5
- rule trace_clearance: 0.2 -> 0.15

Commit message: PCB zamowione
Parts:
- moved R12 13.4 mm to (131.1, 140.7), turned to 180 degrees
- moved R13 13.3 mm to (131.1, 137.6), turned to 180 degrees
- moved R7 12.9 mm to (137.0, 141.3)
- moved J6 12.6 mm to (116.4, 157.0), turned to 90 degrees
- moved R10 12.0 mm to (131.1, 146.8), turned to 180 degrees
- moved R4 11.9 mm to (149.9, 145.2)
- moved L1 9.60 mm to (102.3, 135.1)
- moved R9 8.22 mm to (143.1, 141.4)
- moved R1 7.42 mm to (90.6, 146.4)
- moved R11 7.41 mm to (131.1, 143.7), turned to 180 degrees
- moved R2 7.11 mm to (94.4, 146.5)
- moved R6 7.00 mm to (137.0, 145.2), turned to 180 degrees
- moved R8 6.84 mm to (143.1, 145.2), turned to 180 degrees
- moved C1 6.22 mm to (104.0, 135.1)
- moved C17 5.89 mm to (109.5, 148.7), turned to 180 degrees
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Connections:
- U5 pad 9: (no net) -> PWM_R_IN2
Routing:
- net GND: track 0.00 -> 79.1 mm, vias 0 -> 10
- net PWM_L_IN1: track 24.2 -> 65.3 mm, vias 4 -> 1
- net LED3: track 76.0 -> 38.4 mm, vias 5 -> 1
- net PWM_L_IN2: track 27.7 -> 63.9 mm, vias 3 -> 2
- net +3V3: track 141.2 -> 171.2 mm, vias 8 -> 12
- net LED4: track 65.3 -> 35.9 mm
- net CO_out1: track 68.8 -> 42.2 mm, vias 2 -> 1
- net Net-(C16-Pad1): track 32.9 -> 7.73 mm
- net R_MODE: track 27.3 -> 50.8 mm, vias 3 -> 1
- net L_MODE: track 33.2 -> 56.7 mm, vias 3 -> 1
- net PWM_R_IN1: track 29.7 -> 50.6 mm, vias 4 -> 3
- net CO_enb1: track 55.3 -> 35.1 mm, vias 2 -> 1
- net OUTB_EnkoderL: track 46.4 -> 30.3 mm, vias 0 -> 2
- net SYS_JTCK-SWCLK: track 25.0 -> 39.8 mm, vias 2 -> 1
- net OUTA_EnkoderL: track 50.4 -> 35.9 mm, vias 0 -> 1
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- added copper zone on B.Cu, net GND
- added copper zone on F.Cu, net GND
